File: ChristmasTreePCB/ChristmasTreePCB.kicad_pcb (KiCad board)
At the start: 2 copper layers, 87 x 93.9 mm, 19 parts, among them J1 ICSP, SW1 SPST-NO, U1 ATtiny85-20SHR

Commit message: Updated LED colors and R values. Made BOM
Parts:
- C1: value 0.1 uF -> 0.1 uF 10%
- D1: value White 2V 20mA -> Yellow 2.1V 20mA
- D2, D5: value Green -> Green 2V 20mA
- D3: value Blue -> Red 2V 20mA
- D4, D7: value Red -> Red 2V 20mA
- D6: value Blue -> Green 2V 20mA
- R1, R6: value 10 kohm -> 10 kohm 5%
- R2: value ?? -> 62 ohm 5%
- R3, R4, R5: value ?? -> 33 ohm 5%
Connections:
- net PB2-SCK-BLUE renamed PB2-SCK-DUAL

Commit message: Swap D4 and D6 LED color
Parts:
- C1: value 0.1 uF 10% -> 0.1 uF X7R 20%
- D4: value Red 2V 20mA -> Green 2V 20mA
- D6: value Green 2V 20mA -> Red 2V 20mA
